File: TriacControl.kicad_sch (KiCad schematic)
At the start: 53 parts, among them J1 AC LINE, J2 LOAD, J3 ZEROCROSS, J4 PWM, Q1 BTA16-600, Q2 2N2907, U1 MOC3023, U2 PC817, U3 PC817

Commit message: Added snubber capacitor calculation
Parts:
- R10, R9: value 100R -> 22k
- R11: value 100R -> NC
Changed lines of the file:
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@@
       (effects (font (size 1.27 1.27)) (justify left))
     )
-    (property "Value" "100R" (at 162.56 130.81 90)
+    (property "Value" "22k" (at 162.56 130.175 90)
       (effects (font (size 1.27 1.27)) (justify left))
     )
@@
       (effects (font (size 1.27 1.27)) (justify left))
     )
-    (property "Value" "100R" (at 152.4 130.81 90)
+    (property "Value" "22k" (at 152.4 130.175 90)
       (effects (font (size 1.27 1.27)) (justify left))
     )
@@
       (effects (font (size 1.27 1.27)) (justify left))
     )
-    (property "Value" "100R" (at 157.48 130.81 90)
-      (effects (font (size 1.27 1.27)) (justify left))
-    )
+    (property "Value" "NC" (at 157.48 129.54 90)
+      (effects (font (size 1.27 1.27)) (justify left))
+    )
