File: TriacControl.kicad_pcb (KiCad board)
At the start: 2 copper layers, 100 x 53 mm, 53 parts, among them J1 AC LINE, J2 LOAD, J3 ZEROCROSS, J4 PWM, Q1 BTA16-600, Q2 2N2907, U1 MOC3023, U2 PC817, U3 PC817

Commit message: Updated TRIAC and snubber circuit
Parts:
- C1: value 10 nF, 400 V -> 100 nF, 400 V
- Q1: value BTA16-600 -> BTA24-600B
- R10, R9: value 22k -> 100R
Changed lines of the file:
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@@
         (effects (font (size 1 1) (thickness 0.15)))
     )
-    (fp_text value "10 nF, 400 V" (at 3.75 2.5 -90) (layer "F.Fab")
+    (fp_text value "100 nF, 400 V" (at 3.75 2.5 -90) (layer "F.Fab")
         (effects (font (size 1 1) (thickness 0.15)))
     )
@@
         (effects (font (size 1 1) (thickness 0.15)))
     )
-    (fp_text value "22k" (at 3.81 2.37) (layer "F.Fab")
+    (fp_text value "100R" (at 3.81 2.37) (layer "F.Fab")
         (effects (font (size 1 1) (thickness 0.15)))
     )
@@
         (effects (font (size 1 1) (thickness 0.15)))
     )
-    (fp_text value "BTA16-600" (at 2.54 2.5) (layer "F.Fab")
+    (fp_text value "BTA24-600B" (at 2.54 2.5) (layer "F.Fab")
         (effects (font (size 1 1) (thickness 0.15)))
     )
@@
         (effects (font (size 1 1) (thickness 0.15)))
     )
-    (fp_text value "22k" (at 3.81 2.37) (layer "F.Fab")
-        (effects (font (size 1 1) (thickness 0.15)))
-    )
+    (fp_text value "100R" (at 3.81 2.37) (layer "F.Fab")
+        (effects (font (size 1 1) (thickness 0.15)))
+    )
